File: ESP32WROOM.kicad_sch (KiCad schematic)
At the start: 11 parts, among them J11 ANT2, J14 ESP_ANTENA, SW2 ESP RESET, SW3 ESP BOOT, U2 ESP32-WROOM-32

Commit message: Add files via upload
Parts:
- added D19: LED_TX, LED_SMD:LED_0603_1608Metric, symbol Device:LED
- added R32: 220, Resistor_SMD:R_0603_1608Metric, symbol Device:R_Small
- D18: value LED -> LED_RX
Connections:
- net GND: now also R32.1
- net BOOT-EMAC_REFCLKO renamed BOOT-ETH_REFCLKO
- net EMAC_OSCEN renamed USART1_RX
- net USART1_RX: now also D18.2 (A)
- net IO16 renamed USART1_TX
- net USART1_TX: now also D19.2 (A); no longer D18.2 (A)
- net IO34: no longer names the net of U2.6 (IO34)
- net IO35: no longer names the net of U2.7 (IO35)
- net S_VN: no longer names the net of U2.5 (SENSOR_VN)
- net S_VP: no longer names the net of U2.4 (SENSOR_VP)
- new net: D19.1 (K), R32.2
- no-connect marks 6 -> 10
Other:
- note added: "ESP PROG"
- note added: "ESP-STM"
- note added: "IO1 - UART0_TX"
- note added: "IO16 - UART2_RX"
- note added: "IO17 - UART2_TX"
- note added: "IO3 - UART0_RX"
- note removed: "GPIO"
- note removed: "IO1 - UART_TX"
- note removed: "IO16 - IO"
- note removed: "IO17 - EMAC_OSCEN"
- note removed: "IO3 - UART_RX"
- note removed: "IO34 - IN"
- note removed: "IO35 - IN"
- note removed: "S_VN - IN"
- note removed: "S_VP - IN"
- moved on the sheet: D18, R93

Commit message: Add files via upload
Parts:
- removed U2: ESP32-WROOM-32, RF_Module:ESP32-WROOM-32, symbol RF_Module:ESP32-WROOM-32
- added U2: ESP32-WROOM-32D, RF_Module:ESP32-WROOM-32, symbol RF_Module:ESP32-WROOM-32D
Connections:
- net +3.3V: now also U2.2 (VDD)
- net BOOT-ETH_REFCLKO: now also U2.25 (IO0)
- net EMAC_MDC: now also U2.37 (IO23)
- net EMAC_MDIO: now also U2.30 (IO18)
- net EMAC_RXD0: now also U2.10 (IO25)
- net EMAC_RXD1: now also U2.11 (IO26)
- net EMAC_RX_DV: now also U2.12 (IO27)
- net EMAC_TXD0: now also U2.31 (IO19)
- net EMAC_TXD1: now also U2.36 (IO22)
- net EMAC_TXEN: now also U2.33 (IO21)
- net ESP_I2S_CK: now also U2.8 (IO32)
- net ESP_I2S_SD: now also U2.9 (IO33)
- net ESP_I2S_WS: now also U2.29 (IO5)
- net ESP_RESET: now also U2.3 (EN)
- net ESP_SDIO_CK: now also U2.13 (IO14)
- net ESP_SDIO_CMD: now also U2.23 (IO15)
- net ESP_SDIO_D0: now also U2.24 (IO2)
- net ESP_SDIO_D1: now also U2.26 (IO4)
- net ESP_SDIO_D2: now also U2.14 (IO12)
- net ESP_SDIO_D3: now also U2.16 (IO13)
- net GND: now also U2.1 (GND), U2.15 (GND), U2.38 (GND), U2.39 (GND)
- net RXD0: now also U2.34 (RXD0/IO3)
- net TXD0: now also U2.35 (TXD0/IO1)
- net USART1_RX: now also U2.28 (IO17)
- net USART1_TX: now also U2.27 (IO16)
