File: POWER.kicad_sch (KiCad schematic)
At the start: 64 parts, among them IC1 MP1584EN, IC2 MP1584EN, Q3 QM6006D

Commit message: Add files via upload
Parts:
- added C68, C69: 100nF, Capacitor_SMD:C_0603_1608Metric, symbol Device:C_Small
- added C70, C71: 10uF, Capacitor_SMD:C_1206_3216Metric, symbol Device:C_Small
Connections:
- net +3.3V: now also C68.2, C69.2, C70.2, C71.2
- net GND: now also C68.1, C69.1, C70.1, C71.1
Changed lines of the file:
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@@
   (junction (at 81.28 113.665) (diameter 0) (color 0 0 0 0)
   )
+  (junction (at 187.96 96.52) (diameter 0) (color 0 0 0 0)
+  )
   (junction (at 87.63 36.195) (diameter 0) (color 0 0 0 0)
   )
@@
   (junction (at 147.32 85.09) (diameter 0) (color 0 0 0 0)
   )
+  (junction (at 177.8 96.52) (diameter 0) (color 0 0 0 0)
+  )
   (junction (at 91.44 96.52) (diameter 0) (color 0 0 0 0)
   )
@@
   (junction (at 142.24 85.09) (diameter 0) (color 0 0 0 0)
   )
+  (junction (at 187.96 85.09) (diameter 0) (color 0 0 0 0)
+  )
   (junction (at 40.64 85.09) (diameter 0) (color 0 0 0 0)
   )
@@
   (junction (at 31.75 123.19) (diameter 0) (color 0 0 0 0)
   )
+  (junction (at 182.88 96.52) (diameter 0) (color 0 0 0 0)
+  )
   (junction (at 50.8 96.52) (diameter 0) (color 0 0 0 0)
   )
@@
   (junction (at 137.16 96.52) (diameter 0) (color 0 0 0 0)
   )
+  (junction (at 172.72 85.09) (diameter 0) (color 0 0 0 0)
+  )
   (junction (at 55.88 85.09) (diameter 0) (color 0 0 0 0)
   )
@@
   (junction (at 22.86 85.09) (diameter 0) (color 0 0 0 0)
   )
+  (junction (at 177.8 85.09) (diameter 0) (color 0 0 0 0)
+  )
   (junction (at 76.2 85.09) (diameter 0) (color 0 0 0 0)
   )
@@
   (junction (at 45.72 96.52) (diameter 0) (color 0 0 0 0)
   )
+  (junction (at 172.72 96.52) (diameter 0) (color 0 0 0 0)
+  )
   (junction (at 182.88 36.195) (diameter 0) (color 0 0 0 0)
   )
@@
   (junction (at 120.65 43.815) (diameter 0) (color 0 0 0 0)
   )
+  (junction (at 182.88 85.09) (diameter 0) (color 0 0 0 0)
+  )
   (junction (at 60.96 96.52) (diameter 0) (color 0 0 0 0)
   )
@@
     (stroke (width 0) (type default) (color 0 0 0 0))
   )
+  (wire (pts (xy 187.96 90.17) (xy 187.96 85.09))
+    (stroke (width 0) (type default) (color 0 0 0 0))
+  )
   (wire (pts (xy 140.97 60.325) (xy 140.97 56.515))
     (stroke (width 0) (type default) (color 0 0 0 0))
@@
     (stroke (width 0) (type default) (color 0 0 0 0))
   )
+  (wire (pts (xy 172.72 96.52) (xy 177.8 96.52))
+    (stroke (width 0) (type default) (color 0 0 0 0))
+  )
   (wire (pts (xy 86.36 36.195) (xy 87.63 36.195))
     (stroke (width 0) (type default) (color 0 0 0 0))
@@
     (stroke (width 0) (type default) (color 0 0 0 0))
   )
+  (wire (pts (xy 177.8 96.52) (xy 182.88 96.52))
+    (stroke (width 0) (type default) (color 0 0 0 0))
+  )
   (wire (pts (xy 50.8 85.09) (xy 55.88 85.09))
     (stroke (width 0) (type default) (color 0 0 0 0))
@@
     (stroke (width 0) (type default) (color 0 0 0 0))
   )
+  (wire (pts (xy 187.96 85.09) (xy 182.88 85.09))
+    (stroke (width 0) (type default) (color 0 0 0 0))
+  )
   (wire (pts (xy 101.6 95.25) (xy 101.6 96.52))
     (stroke (width 0) (type default) (color 0 0 0 0))
@@
     (stroke (width 0) (type default) (color 0 0 0 0))
   )
+  (wire (pts (xy 172.72 85.09) (xy 177.8 85.09))
+    (stroke (width 0) (type default) (color 0 0 0 0))
+  )
   (wire (pts (xy 137.16 96.52) (xy 137.16 95.25))
     (stroke (width 0) (type default) (color 0 0 0 0))
@@
     (stroke (width 0) (type default) (color 0 0 0 0))
   )
+  (wire (pts (xy 177.8 85.09) (xy 177.8 90.17))
+    (stroke (width 0) (type default) (color 0 0 0 0))
+  )
   (wire (pts (xy 76.2 85.09) (xy 78.74 85.09))
     (stroke (width 0) (type default) (color 0 0 0 0))
@@
     (stroke (width 0) (type default) (color 0 0 0 0))
   )
+  (wire (pts (xy 182.88 96.52) (xy 182.88 95.25))
+    (stroke (width 0) (type default) (color 0 0 0 0))
+  )
   (wire (pts (xy 50.8 60.325) (xy 50.8 56.515))
     (stroke (width 0) (type default) (color 0 0 0 0))
@@
     (stroke (width 0) (type default) (color 0 0 0 0))
   )
+  (wire (pts (xy 187.96 95.25) (xy 187.96 96.52))
+    (stroke (width 0) (type default) (color 0 0 0 0))
+  )
   (wire (pts (xy 182.88 42.545) (xy 182.88 55.245))
     (stroke (width 0) (type default) (color 0 0 0 0))
@@
     (stroke (width 0) (type default) (color 0 0 0 0))
   )
+  (wire (pts (xy 187.96 96.52) (xy 182.88 96.52))
+    (stroke (width 0) (type default) (color 0 0 0 0))
+  )
   (wire (pts (xy 91.44 96.52) (xy 91.44 95.25))
     (stroke (width 0) (type default) (color 0 0 0 0))
@@
     (stroke (width 0) (type default) (color 0 0 0 0))
   )
+  (wire (pts (xy 193.04 85.09) (xy 187.96 85.09))
+    (stroke (width 0) (type default) (color 0 0 0 0))
+  )
   (wire (pts (xy 172.72 36.195) (xy 158.75 36.195))
     (stroke (width 0) (type default) (color 0 0 0 0))
@@
     (stroke (width 0) (type default) (color 0 0 0 0))
   )
+  (wire (pts (xy 193.04 95.25) (xy 193.04 96.52))
+    (stroke (width 0) (type default) (color 0 0 0 0))
+  )
+  (wire (pts (xy 182.88 85.09) (xy 182.88 90.17))
+    (stroke (width 0) (type default) (color 0 0 0 0))
+  )
   (wire (pts (xy 116.84 96.52) (xy 121.92 96.52))
     (stroke (width 0) (type default) (color 0 0 0 0))
@@
     (stroke (width 0) (type default) (color 0 0 0 0))
   )
+  (wire (pts (xy 177.8 95.25) (xy 177.8 96.52))
+    (stroke (width 0) (type default) (color 0 0 0 0))
+  )
   (wire (pts (xy 33.02 36.195) (xy 25.4 36.195))
     (stroke (width 0) (type default) (color 0 0 0 0))
@@
     (stroke (width 0) (type default) (color 0 0 0 0))
   )
+  (wire (pts (xy 193.04 90.17) (xy 193.04 85.09))
+    (stroke (width 0) (type default) (color 0 0 0 0))
+  )
   (wire (pts (xy 128.27 42.545) (xy 125.73 42.545))
     (stroke (width 0) (type default) (color 0 0 0 0))
@@
     (stroke (width 0) (type default) (color 0 0 0 0))
   )
+  (wire (pts (xy 193.04 96.52) (xy 187.96 96.52))
+    (stroke (width 0) (type default) (color 0 0 0 0))
+  )
   (wire (pts (xy 64.77 50.165) (xy 64.77 48.895))
     (stroke (width 0) (type default) (color 0 0 0 0))
@@
   )
   (wire (pts (xy 111.76 95.25) (xy 111.76 96.52))
+    (stroke (width 0) (type default) (color 0 0 0 0))
+  )
+  (wire (pts (xy 177.8 85.09) (xy 182.88 85.09))
     (stroke (width 0) (type default) (color 0 0 0 0))
   )
@@
     )
     (property "Datasheet" "~" (id 3) (at 127 57.785 0)
+      (effects (font (size 1.27 1.27)) hide)
+    )
+    (pin "1")
+    (pin "2")
+  )
+  (symbol (lib_id "Device:C_Small") (at 182.88 92.71 0) (mirror x) (unit 1)
+    (in_bom yes) (on_board yes)
+    (property "Reference" "C69" (id 0) (at 185.42 93.98 90))
+    (property "Value" "100nF" (id 1) (at 185.42 88.9 90))
+    (property "Footprint" "Capacitor_SMD:C_0603_1608Metric" (id 2) (at 182.88 92.71 0)
+      (effects (font (size 1.27 1.27)) hide)
+    )
+    (property "Datasheet" "~" (id 3) (at 182.88 92.71 0)
       (effects (font (size 1.27 1.27)) hide)
     )
@@
     (pin "2")
   )
+  (symbol (lib_id "Device:C_Small") (at 193.04 92.71 0) (mirror x) (unit 1)
+    (in_bom yes) (on_board yes)
+    (property "Reference" "C71" (id 0) (at 195.58 93.98 90))
+    (property "Value" "10uF" (id 1) (at 195.58 88.9 90))
+    (property "Footprint" "Capacitor_SMD:C_1206_3216Metric" (id 2) (at 193.04 92.71 0)
+      (effects (font (size 1.27 1.27)) hide)
+    )
+    (property "Datasheet" "~" (id 3) (at 193.04 92.71 0)
+      (effects (font (size 1.27 1.27)) hide)
+    )
+    (pin "1")
+    (pin "2")
+  )
   (symbol (lib_id "Device:C_Small") (at 152.4 27.305 90) (unit 1)
     (in_bom yes) (on_board yes)
@@
     )
     (pin "1")
+  )
+  (symbol (lib_id "Device:C_Small") (at 177.8 92.71 0) (mirror x) (unit 1)
+    (in_bom yes) (on_board yes)
+    (property "Reference" "C68" (id 0) (at 180.34 93.98 90))
+    (property "Value" "100nF" (id 1) (at 180.34 88.9 90))
+    (property "Footprint" "Capacitor_SMD:C_0603_1608Metric" (id 2) (at 177.8 92.71 0)
+      (effects (font (size 1.27 1.27)) hide)
+    )
+    (property "Datasheet" "~" (id 3) (at 177.8 92.71 0)
+      (effects (font (size 1.27 1.27)) hide)
+    )
+    (pin "1")
+    (pin "2")
   )
   (symbol (lib_id "power:GND") (at 50.8 60.325 0) (unit 1)
@@
     (pin "9")
   )
+  (symbol (lib_id "Device:C_Small") (at 187.96 92.71 0) (mirror x) (unit 1)
+    (in_bom yes) (on_board yes)
+    (property "Reference" "C70" (id 0) (at 190.5 93.98 90))
+    (property "Value" "10uF" (id 1) (at 190.5 88.9 90))
+    (property "Footprint" "Capacitor_SMD:C_1206_3216Metric" (id 2) (at 187.96 92.71 0)
+      (effects (font (size 1.27 1.27)) hide)
+    )
+    (property "Datasheet" "~" (id 3) (at 187.96 92.71 0)
+      (effects (font (size 1.27 1.27)) hide)
+    )
+    (pin "1")
+    (pin "2")
+  )
   (symbol (lib_id "MP1584EN-LF-P:MP1584EN") (at 48.26 42.545 0) (unit 1)
