File: TFT_LCD.kicad_sch (KiCad schematic)
At the start: 2 parts, among them J3 FPC_32p

Commit message: Add files via upload
Parts:
- added R31: 100, Resistor_SMD:R_0805_2012Metric, symbol Device:R_Small
Connections:
- net +3.3V: no longer J3.29
- new net: J3.29, R31.1
- new net +5V: R31.2
Changed lines of the file:
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@@
     (pin "1")
+  )
+  (symbol (lib_id "Device:R_Small") (at 73.66 116.84 270) (unit 1)
+    (in_bom yes) (on_board yes)
+    (property "Reference" "R31" (id 0) (at 69.85 115.57 90))
+    (property "Value" "100" (id 1) (at 73.66 116.84 90))
+    (property "Footprint" "Resistor_SMD:R_0805_2012Metric" (id 2) (at 73.66 116.84 0)
+      (effects (font (size 1.27 1.27)) hide)
+    )
+    (property "Datasheet" "~" (id 3) (at 73.66 116.84 0)
+      (effects (font (size 1.27 1.27)) hide)
+    )
+    (pin "1")
+    (pin "2")
   )
   (symbol (lib_id "power:GND") (at 76.2 48.26 270) (mirror x) (unit 1)
@@
     (pin "1")
   )
-  (symbol (lib_id "power:+3.3V") (at 76.2 116.84 90) (mirror x) (unit 1)
-    (in_bom yes) (on_board yes)
-    (property "Reference" "#PWR048" (id 0) (at 80.01 116.84 0)
-      (effects (font (size 1.27 1.27)) hide)
-    )
-    (property "Value" "+3.3V" (id 1) (at 69.85 116.84 90))
-    (property "Footprint" "" (id 2) (at 76.2 116.84 0)
-      (effects (font (size 1.27 1.27)) hide)
-    )
-    (property "Datasheet" "" (id 3) (at 76.2 116.84 0)
-      (effects (font (size 1.27 1.27)) hide)
-    )
-    (pin "1")
-  )
   (symbol (lib_id "power:GND") (at 76.2 121.92 270) (mirror x) (unit 1)
     (in_bom yes) (on_board yes)
@@
       (effects (font (size 1.27 1.27)) hide)
     )
+    (pin "1")
+  )
+  (symbol (lib_id "power:+5V") (at 71.12 116.84 90) (unit 1)
+    (in_bom yes) (on_board yes)
+    (property "Reference" "#PWR0163" (id 0) (at 74.93 116.84 0)
+      (effects (font (size 1.27 1.27)) hide)
+    )
+    (property "Value" "+5V" (id 1) (at 67.945 116.84 90)
+      (effects (font (size 1.27 1.27)) (justify left))
+    )
+    (property "Footprint" "" (id 2) (at 71.12 116.84 0)
+      (effects (font (size 1.27 1.27)) hide)
+    )
+    (property "Datasheet" "" (id 3) (at 71.12 116.84 0)
+      (effects (font (size 1.27 1.27)) hide)
+    )
