File: CONNECTOR.kicad_sch (KiCad schematic)
At the start: 11 parts, among them J10 SWD, J2 STM_IO, J7 CONNECTOR

Commit message: Add files via upload
Connections:
- net GND: now also J7.14 (Pin_14); no longer J7.16 (Pin_16)
- net RS485_A: now also J7.16 (Pin_16); no longer J7.15 (Pin_15)
- net RS485_B: now also J7.15 (Pin_15); no longer J7.14 (Pin_14)
Changed lines of the file:
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@@
     )
   )
-  (global_label "RS485_A" (shape bidirectional) (at 71.12 95.885 180) (fields_autoplaced)
-    (effects (font (size 1.27 1.27)) (justify right))
-    (property "Intersheet References" "${INTERSHEET_REFS}" (id 0) (at 60.5426 95.9644 0)
+  (global_label "RS485_A" (shape bidirectional) (at 71.12 98.425 180) (fields_autoplaced)
+    (effects (font (size 1.27 1.27)) (justify right))
+    (property "Intersheet References" "${INTERSHEET_REFS}" (id 0) (at 60.5426 98.5044 0)
       (effects (font (size 1.27 1.27)) (justify right) hide)
     )
@@
     )
   )
-  (global_label "RS485_B" (shape bidirectional) (at 71.12 93.345 180) (fields_autoplaced)
-    (effects (font (size 1.27 1.27)) (justify right))
-    (property "Intersheet References" "${INTERSHEET_REFS}" (id 0) (at 60.3612 93.4244 0)
+  (global_label "RS485_B" (shape bidirectional) (at 71.12 95.885 180) (fields_autoplaced)
+    (effects (font (size 1.27 1.27)) (justify right))
+    (property "Intersheet References" "${INTERSHEET_REFS}" (id 0) (at 60.3612 95.9644 0)
       (effects (font (size 1.27 1.27)) (justify right) hide)
     )
@@
     (pin "1")
   )
-  (symbol (lib_id "power:GND") (at 71.12 98.425 270) (unit 1)
-    (in_bom yes) (on_board yes)
-    (property "Reference" "#PWR0165" (id 0) (at 64.77 98.425 0)
-      (effects (font (size 1.27 1.27)) hide)
-    )
-    (property "Value" "GND" (id 1) (at 67.31 98.425 90)
-      (effects (font (size 1.27 1.27)) (justify right))
-    )
-    (property "Footprint" "" (id 2) (at 71.12 98.425 0)
-      (effects (font (size 1.27 1.27)) hide)
-    )
-    (property "Datasheet" "" (id 3) (at 71.12 98.425 0)
-      (effects (font (size 1.27 1.27)) hide)
-    )
+  (symbol (lib_id "power:GND") (at 71.12 93.345 270) (unit 1)
+    (in_bom yes) (on_board yes)
+    (property "Reference" "#PWR0165" (id 0) (at 64.77 93.345 0)
+      (effects (font (size 1.27 1.27)) hide)
+    )
+    (property "Value" "GND" (id 1) (at 67.31 93.345 90)
+      (effects (font (size 1.27 1.27)) (justify right))
+    )
+    (property "Footprint" "" (id 2) (at 71.12 93.345 0)
+      (effects (font (size 1.27 1.27)) hide)
+    )
+    (property "Datasheet" "" (id 3) (at 71.12 93.345 0)
+      (effects (font (size 1.27 1.27)) hide)
+    )
