File: RTC.kicad_sch (KiCad schematic)
At the start: 4 parts, among them J8 BAT, U7 DS3231M

Commit message: Add files via upload
Parts:
- removed R87: 1k, Resistor_SMD:R_0603_1608Metric, symbol Device:R_Small
- added D21: 1N4007, Diode_SMD:D_SOD-123F, symbol Diode:PMEG3010EH
Connections:
- net +3.3V: now also D21.2 (A); no longer D17.2 (A), U7.2 (VCC)
- net at J8.1 (Pin_1): now also D17.2 (A); no longer D17.1 (K)
- net at U7.14 (VBAT): now also D17.1 (K)
- new net: D21.1 (K), U7.2 (VCC)
Other:
- moved on the sheet: D17, J8
Changed lines of the file:
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@@
 (kicad_sch (version 20211123) (generator eeschema)
   (paper "A5")
-  (junction (at 107.315 53.975) (diameter 0) (color 0 0 0 0)
-  )
   (no_connect (at 78.74 70.485))
   (no_connect (at 104.14 67.945))
   (no_connect (at 104.14 60.325))
-  (wire (pts (xy 113.665 53.975) (xy 109.855 53.975))
+  (wire (pts (xy 107.95 53.975) (xy 104.14 53.975))
     (stroke (width 0) (type default) (color 0 0 0 0))
   )
@@
     (stroke (width 0) (type default) (color 0 0 0 0))
   )
-  (wire (pts (xy 91.44 53.975) (xy 95.25 53.975))
+  (wire (pts (xy 91.44 53.975) (xy 92.71 53.975))
     (stroke (width 0) (type default) (color 0 0 0 0))
   )
-  (wire (pts (xy 109.855 53.975) (xy 109.855 52.705))
+  (wire (pts (xy 104.14 53.975) (xy 104.14 52.705))
     (stroke (width 0) (type default) (color 0 0 0 0))
   )
-  (wire (pts (xy 100.33 53.975) (xy 107.315 53.975))
+  (wire (pts (xy 100.33 53.975) (xy 101.6 53.975))
     (stroke (width 0) (type default) (color 0 0 0 0))
   )
-  (wire (pts (xy 107.315 53.975) (xy 107.315 55.245))
-    (stroke (width 0) (type default) (color 0 0 0 0))
-  )
-  (wire (pts (xy 107.315 52.705) (xy 107.315 53.975))
+  (wire (pts (xy 101.6 52.705) (xy 101.6 53.975))
     (stroke (width 0) (type default) (color 0 0 0 0))
   )
@@
     )
   )
-  (symbol (lib_id "power:GND") (at 113.665 53.975 90) (unit 1)
+  (symbol (lib_id "Diode:PMEG3010EH") (at 88.9 51.435 90) (unit 1)
     (in_bom yes) (on_board yes)
-    (property "Reference" "#PWR039" (id 0) (at 120.015 53.975 0)
+    (property "Reference" "D21" (id 0) (at 84.455 51.435 0))
+    (property "Value" "1N4007" (id 1) (at 86.36 51.435 0))
+    (property "Footprint" "Diode_SMD:D_SOD-123F" (id 2) (at 93.345 51.435 0)
       (effects (font (size 1.27 1.27)) hide)
     )
-    (property "Value" "GND" (id 1) (at 118.745 53.975 90))
-    (property "Footprint" "" (id 2) (at 113.665 53.975 0)
-      (effects (font (size 1.27 1.27)) hide)
-    )
-    (property "Datasheet" "" (id 3) (at 113.665 53.975 0)
-      (effects (font (size 1.27 1.27)) hide)
-    )
-    (pin "1")
-  )
-  (symbol (lib_id "Connector:Conn_01x02_Male") (at 107.315 47.625 90) (mirror x) (unit 1)
-    (in_bom yes) (on_board yes) (fields_autoplaced)
-    (property "Reference" "J8" (id 0) (at 111.76 46.9899 90)
-      (effects (font (size 1.27 1.27)) (justify right))
-    )
-    (property "Value" "BAT" (id 1) (at 111.76 49.5299 90)
-      (effects (font (size 1.27 1.27)) (justify right))
-    )
-    (property "Footprint" "XH_2.54mm_Conn:XH_2P_2.54mm_Vertical" (id 2) (at 107.315 47.625 0)
-      (effects (font (size 1.27 1.27)) hide)
-    )
-    (property "Datasheet" "~" (id 3) (at 107.315 47.625 0)
+    (property "Datasheet" "https://assets.nexperia.com/documents/data-sheet/PMEG3010EH_EJ_ET.pdf" (id 3) (at 88.9 51.435 0)
       (effects (font (size 1.27 1.27)) hide)
     )
@@
     (pin "2")
   )
-  (symbol (lib_id "Device:R_Small") (at 97.79 53.975 90) (unit 1)
+  (symbol (lib_id "power:GND") (at 107.95 53.975 90) (unit 1)
     (in_bom yes) (on_board yes)
-    (property "Reference" "R87" (id 0) (at 97.79 50.165 90))
-    (property "Value" "1k" (id 1) (at 97.79 52.07 90))
-    (property "Footprint" "Resistor_SMD:R_0603_1608Metric" (id 2) (at 97.79 53.975 0)
+    (property "Reference" "#PWR039" (id 0) (at 114.3 53.975 0)
       (effects (font (size 1.27 1.27)) hide)
     )
-    (property "Datasheet" "~" (id 3) (at 97.79 53.975 0)
+    (property "Value" "GND" (id 1) (at 113.03 53.975 90))
+    (property "Footprint" "" (id 2) (at 107.95 53.975 0)
+      (effects (font (size 1.27 1.27)) hide)
+    )
+    (property "Datasheet" "" (id 3) (at 107.95 53.975 0)
+      (effects (font (size 1.27 1.27)) hide)
+    )
+    (pin "1")
+  )
+  (symbol (lib_id "Connector:Conn_01x02_Male") (at 101.6 47.625 90) (mirror x) (unit 1)
+    (in_bom yes) (on_board yes) (fields_autoplaced)
+    (property "Reference" "J8" (id 0) (at 106.045 46.9899 90)
+      (effects (font (size 1.27 1.27)) (justify right))
+    )
+    (property "Value" "BAT" (id 1) (at 106.045 49.5299 90)
+      (effects (font (size 1.27 1.27)) (justify right))
+    )
+    (property "Footprint" "XH_2.54mm_Conn:XH_2P_2.54mm_Vertical" (id 2) (at 101.6 47.625 0)
+      (effects (font (size 1.27 1.27)) hide)
+    )
+    (property "Datasheet" "~" (id 3) (at 101.6 47.625 0)
       (effects (font (size 1.27 1.27)) hide)
     )
@@
     (pin "9")
   )
-  (symbol (lib_id "Diode:PMEG3010EH") (at 107.315 59.055 270) (unit 1)
+  (symbol (lib_id "Diode:PMEG3010EH") (at 96.52 53.975 0) (unit 1)
     (in_bom yes) (on_board yes)
-    (property "Reference" "D17" (id 0) (at 111.76 59.055 0))
-    (property "Value" "1N4007" (id 1) (at 109.855 59.055 0))
-    (property "Footprint" "Diode_SMD:D_SOD-123F" (id 2) (at 102.87 59.055 0)
+    (property "Reference" "D17" (id 0) (at 96.52 49.53 0))
+    (property "Value" "1N4007" (id 1) (at 96.52 51.435 0))
+    (property "Footprint" "Diode_SMD:D_SOD-123F" (id 2) (at 96.52 58.42 0)
       (effects (font (size 1.27 1.27)) hide)
     )
-    (property "Datasheet" "https://assets.nexperia.com/documents/data-sheet/PMEG3010EH_EJ_ET.pdf" (id 3) (at 107.315 59.055 0)
+    (property "Datasheet" "https://assets.nexperia.com/documents/data-sheet/PMEG3010EH_EJ_ET.pdf" (id 3) (at 96.52 53.975 0)
       (effects (font (size 1.27 1.27)) hide)
     )
@@
     (pin "1")
   )
-  (symbol (lib_id "power:+3.3V") (at 88.9 55.245 0) (unit 1)
+  (symbol (lib_id "power:+3.3V") (at 88.9 47.625 0) (unit 1)
     (in_bom yes) (on_board yes)
-    (property "Reference" "#PWR037" (id 0) (at 88.9 59.055 0)
+    (property "Reference" "#PWR037" (id 0) (at 88.9 51.435 0)
       (effects (font (size 1.27 1.27)) hide)
     )
-    (property "Value" "+3.3V" (id 1) (at 88.9 51.435 0))
-    (property "Footprint" "" (id 2) (at 88.9 55.245 0)
+    (property "Value" "+3.3V" (id 1) (at 88.9 43.815 0))
+    (property "Footprint" "" (id 2) (at 88.9 47.625 0)
       (effects (font (size 1.27 1.27)) hide)
     )
-    (property "Datasheet" "" (id 3) (at 88.9 55.245 0)
+    (property "Datasheet" "" (id 3) (at 88.9 47.625 0)
       (effects (font (size 1.27 1.27)) hide)
     )
-    (pin "1")
-  )
-  (symbol (lib_id "power:+3.3V") (at 107.315 62.865 180) (unit 1)
-    (in_bom yes) (on_board yes)
-    (property "Reference" "#PWR0156" (id 0) (at 107.315 59.055 0)
-      (effects (font (size 1.27 1.27)) hide)
-    )
-    (property "Value" "+3.3V" (id 1) (at 107.315 66.675 0))
-    (property "Footprint" "" (id 2) (at 107.315 62.865 0)
-      (effects (font (size 1.27 1.27)) hide)
-    )
-    (property "Datasheet" "" (id 3) (at 107.315 62.865 0)
-      (effects (font (size 1.27 1.27)) hide)
-    )
